File: rgb_led_pcb/rgb_led_pcb.kicad_pcb (KiCad board)
At the start: 2 copper layers, 33 x 33 mm, 11 parts

Commit message: updated
Parts:
- added G***: LOGO, MyLibrary:nitkc_logo, B.Cu at (56.5, 56.5)

Commit message: updated
Parts:
- moved R1 15.0 mm to (50.0, 57.0)
- moved R2 15.0 mm to (50.0, 60.5)
- moved USB-C 10.5 mm to (43.6, 46.0)
Routing:
- net +5V: track 73.7 -> 11.5 mm
- net Net-(LED3-Pad2): track 31.4 -> 0.00 mm
- net Net-(LED1-Pad2): track 25.5 -> 0.00 mm
- net Net-(LED2-Pad2): track 20.4 -> 0.18 mm
- net Net-(J1-PadB5): track 18.6 -> 0.00 mm
- net unconnected-(J1-PadS1): track 16.2 -> 0.00 mm
- net Net-(R5-Pad1): track 14.5 -> 0.00 mm
- net Net-(R3-Pad1): track 14.5 -> 0.00 mm
- net Net-(R4-Pad1): track 14.3 -> 0.00 mm
- net Net-(J1-PadA5): track 13.0 -> 0.00 mm
- net GND: track 54.2 -> 43.5 mm
- removed copper zone on F.Cu, net +5V
- removed copper zone on B.Cu, net GND
Other:
- board text removed: "National Institute of Technology Kagawa College Designed by MILab"
